File: Pixel-Interface-Board/Pixel-Interface-Board.sch (KiCad schematic (older format))
At the start: 29 parts, among them IC1 ATTINY85-P, P1 CONN_20X2, SW1 SW_PUSH, SW10 SW_PUSH, SW11 SW_PUSH, SW12 SW_PUSH, SW2 SW_PUSH, SW3 SW_PUSH, SW4 SW_PUSH, SW5 SW_PUSH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

Commit message: Almost done with the Front Board!
Parts:
- removed P1: CONN_20X2, symbol CONN_20X2
- added P1: CONN_02X20, Pin_Headers:Pin_Header_Straight_2x20, symbol CONN_02X20
- D1: footprint ~ -> LEDs:LED-5MM
- IC1: footprint DIP8 -> Housings_DIP:DIP-8_W7.62mm
- R1, R10, R11, R12, R14, R2, R3, R4, R5, R6, R7, R8, R9: footprint ~ -> Resistors_ThroughHole:Resistor_Horizontal_RM10mm
- R13: value R -> 1K; footprint ~ -> Resistors_ThroughHole:Resistor_Horizontal_RM10mm
- SW1, SW10, SW11, SW4, SW7, SW8: footprint ~ -> Buttons_Switches_ThroughHole:SW_PUSH-12mm
- SW12, SW3, SW6, SW9: footprint ~ -> Buttons_Switches_ThroughHole:SW_PUSH_SMALL
- SW2, SW5: footprint ~ -> Buttons_Switches_SMD:SW_SPST_PTS645
Connections:
- wire segments 68 -> 97
- no-connect marks 18 -> 19

Commit message: Fixed the interface board, FINALLY.
Parts:
- SW1, SW10, SW11, SW4, SW7, SW8: footprint Buttons_Switches_ThroughHole:SW_PUSH-12mm -> Buttons_Switches_ThroughHole:SW_PUSH_SMALL
- SW2, SW5: footprint Buttons_Switches_SMD:SW_SPST_PTS645 -> Buttons_Switches_ThroughHole:SW_PUSH_SMALL
Changed lines of the file:
@@
 LIBS:contrib
 LIBS:valves
+LIBS:Pixel-Interface-Board-cache
 EELAYER 25 0
 EELAYER END
@@
 F 0 "SW1" H 2050 5510 50  0000 C CNN
 F 1 "SW_PUSH" H 1900 5320 50  0000 C CNN
-F 2 "Buttons_Switches_ThroughHole:SW_PUSH-12mm" H 1900 5400 60  0001 C CNN
+F 2 "Buttons_Switches_ThroughHole:SW_PUSH_SMALL" H 1900 5400 60  0001 C CNN
 F 3 "~" H 1900 5400 60  0000 C CNN
 	1    1900 5400
@@
 F 0 "SW4" H 2900 5510 50  0000 C CNN
 F 1 "SW_PUSH" H 2750 5320 50  0000 C CNN
-F 2 "Buttons_Switches_ThroughHole:SW_PUSH-12mm" H 2750 5400 60  0001 C CNN
+F 2 "Buttons_Switches_ThroughHole:SW_PUSH_SMALL" H 2750 5400 60  0001 C CNN
 F 3 "~" H 2750 5400 60  0000 C CNN
 	1    2750 5400
@@
 F 0 "SW7" H 3750 5510 50  0000 C CNN
 F 1 "SW_PUSH" H 3600 5320 50  0000 C CNN
-F 2 "Buttons_Switches_ThroughHole:SW_PUSH-12mm" H 3600 5400 60  0001 C CNN
+F 2 "Buttons_Switches_ThroughHole:SW_PUSH_SMALL" H 3600 5400 60  0001 C CNN
 F 3 "~" H 3600 5400 60  0000 C CNN
 	1    3600 5400
@@
 F 0 "SW10" H 4600 5510 50  0000 C CNN
 F 1 "SW_PUSH" H 4450 5320 50  0000 C CNN
-F 2 "Buttons_Switches_ThroughHole:SW_PUSH-12mm" H 4450 5400 60  0001 C CNN
+F 2 "Buttons_Switches_ThroughHole:SW_PUSH_SMALL" H 4450 5400 60  0001 C CNN
 F 3 "~" H 4450 5400 60  0000 C CNN
 	1    4450 5400
@@
 F 0 "SW2" H 2050 6410 50  0000 C CNN
 F 1 "SW_PUSH" H 1900 6220 50  0000 C CNN
-F 2 "Buttons_Switches_SMD:SW_SPST_PTS645" H 1900 6300 60  0001 C CNN
+F 2 "Buttons_Switches_ThroughHole:SW_PUSH_SMALL" H 1900 6300 60  0001 C CNN
 F 3 "~" H 1900 6300 60  0000 C CNN
 	1    1900 6300
@@
 F 0 "SW5" H 2900 6410 50  0000 C CNN
 F 1 "SW_PUSH" H 2750 6220 50  0000 C CNN
-F 2 "Buttons_Switches_SMD:SW_SPST_PTS645" H 2750 6300 60  0001 C CNN
+F 2 "Buttons_Switches_ThroughHole:SW_PUSH_SMALL" H 2750 6300 60  0001 C CNN
 F 3 "~" H 2750 6300 60  0000 C CNN
 	1    2750 6300
@@
 F 0 "SW8" H 3750 6410 50  0000 C CNN
 F 1 "SW_PUSH" H 3600 6220 50  0000 C CNN
-F 2 "Buttons_Switches_ThroughHole:SW_PUSH-12mm" H 3600 6300 60  0001 C CNN
+F 2 "Buttons_Switches_ThroughHole:SW_PUSH_SMALL" H 3600 6300 60  0001 C CNN
 F 3 "~" H 3600 6300 60  0000 C CNN
 	1    3600 6300
@@
 F 0 "SW11" H 4600 6410 50  0000 C CNN
 F 1 "SW_PUSH" H 4450 6220 50  0000 C CNN
-F 2 "Buttons_Switches_ThroughHole:SW_PUSH-12mm" H 4450 6300 60  0001 C CNN
+F 2 "Buttons_Switches_ThroughHole:SW_PUSH_SMALL" H 4450 6300 60  0001 C CNN
 F 3 "~" H 4450 6300 60  0000 C CNN
 	1    4450 6300
